Commit message: Update: cleanup

File: src/control_robot/urdf/2dof.urdf (robot description, URDF)
Before this commit: robot 2dof, 3 links, 2 joints
Links:
- added link ee_link; collision sphere radius=0.05; visual sphere radius=0.05
- link base_link: geometry collision box size=0.2 0.2 0.05; visual box size=0.2 0.2 0.05
- link link1: geometry collision box size=1.0 0.05 0.05; visual box size=1.0 0.05 0.05
- link link2: geometry collision box size=1.0 0.05 0.05; visual box size=1.0 0.05 0.05
Joints:
- added joint ee_fixed: type fixed, parent link2, child ee_link, origin xyz=1.0 0 0 rpy=0 0 0
